Commit message: Rebase from 'upstream'

File: robots/xpp_hyq/urdf/hyq.urdf.xacro (robot description, xacro)
@@ -1,10 +1,9 @@
 <?xml version="1.0"?>
 <robot name="hyq" xmlns:xacro="http://www.ros.org/wiki/xacro">
-  <property name="PI" value="3.1415926535897931"/>
-  - <!-- standard distances -->
-- <property name="d_lr" value="0.414"/>
-- <property name="d_fh" value="0.747"/>
-- <property name="d_tbb" value="0.082"/>
-- <property name="d_p1p2" value="0.35"/>
+  <xacro:property name="PI" value="3.1415926535897931"/>
+  <xacro:property name="d_lr" value="0.414"/>
+  <xacro:property name="d_fh" value="0.747"/>
+  <xacro:property name="d_tbb" value="0.082"/>
+  <xacro:property name="d_p1p2" value="0.35"/>
 	<!-- HyQ trunk -->
 	<xacro:include filename="$(find xpp_hyq)/urdf/trunk.urdf.xacro"/>
@@ -12,9 +11,6 @@
 	<xacro:include filename="$(find xpp_hyq)/urdf/leg.urdf.xacro"/>
 	<!-- Using the macros defined above -->
-	<!-- body -->
 	<!-- trunk -->
-	<xacro:hyq_trunk name="base">
-		<origin xyz="-0.443 -0.191 -0.276" rpy="0 0 0"/>
-	</xacro:hyq_trunk>
+	<xacro:hyq_trunk name="base"/>
 	<!-- LF leg -->
 	<xacro:hyq_leg

File: robots/xpp_hyq/urdf/leg.urdf.xacro (robot description, xacro)
@@ -1,11 +1,10 @@
 <?xml version="1.0"?>
 <robot xmlns:xacro="http://www.ros.org/wiki/xacro">
-	<!-- ================================== Leg ================================== -->
-	<!-- The xacro macro xacro:hyq_leg contains: hip assembly, upper and lower leg -->
+	<!-- leg macro definiction -->
 	<xacro:macro name="hyq_leg" params="name parent *origin reflect_hip reflect_upper reflect_front">
 		<!-- Joints -->
 		<!-- Hip assembly joint -->
 		<joint name="${name}_haa_joint" type="revolute">
-			<insert_block name="origin"/>
+			<xacro:insert_block name="origin"/>
 			<parent link="${parent}"/>
 			<child  link="${name}_hipassembly"/>
@@ -32,6 +31,6 @@
           lower="${-(1+reflect_front)*7*PI/18+(1-reflect_front)*PI/18}"
           upper="${(1-reflect_front)*7*PI/18-(1+reflect_front)*PI/18}"/>
+		</joint>
 		<!-- Foot joint -->
-		</joint>
 		<joint name="${name}_foot_joint" type="fixed">
 			<origin xyz="0.35 0 0" rpy="${PI/2} 0 ${-PI/2}"/>

File: robots/xpp_hyq/urdf/trunk.urdf.xacro (robot description, xacro)
@@ -1,6 +1,5 @@
 <?xml version="1.0"?>
 <robot xmlns:xacro="http://www.ros.org/wiki/xacro">
-	<!-- ================================ Trunk ================================ -->
-	<!-- The xacro macro xacro:hyq_base contains: base and trunk -->
+	<!-- trunk macro definition -->
 	<xacro:macro name="hyq_trunk" params="name">
 		<!-- Floating-base Joint -->
@@ -10,5 +9,4 @@
 			<child link="trunk"/>
 		</joint>
-		<!-- Links -->
 		<!-- Footprint link -->
 		<link name="${name}">
